Commit message: final

File: src/line_bot_description/urdf/robot.urdf (robot description, URDF)
Before this commit: robot giant_line_follower, 8 links, 7 joints
Links:
- removed link sonar_front_link
- added link caster_rear, mass 0.5; collision sphere radius=0.05; visual sphere radius=0.05
- added link sonar_left_link; visual box size=0.05 0.05 0.05
- added link sonar_right_link; visual box size=0.05 0.05 0.05
- link base_link: mass 10.0 -> 20.0; geometry collision box size=1.0 0.6 0.2; visual box size=1.0 0.6 0.2
- link left_wheel: geometry collision cylinder length=0.1 radius=0.15; visual cylinder length=0.1 radius=0.15
- link line_sensor_left: geometry visual box size=0.02 0.02 0.02
- link line_sensor_right: geometry visual box size=0.02 0.02 0.02
- link right_wheel: geometry collision cylinder length=0.1 radius=0.15; visual cylinder length=0.1 radius=0.15
Joints:
- removed joint sonar_front_joint
- added joint caster_rear_joint: type fixed, parent base_link, child caster_rear, origin xyz=-0.4 0 -0.10
- added joint sonar_left_joint: type fixed, parent base_link, child sonar_left_link, origin xyz=0.5 0.2 0.1
- added joint sonar_right_joint: type fixed, parent base_link, child sonar_right_link, origin xyz=0.5 -0.2 0.1
- joint caster_front_joint: origin xyz=0.3 0 -0.10 -> xyz=0.4 0 -0.10
- joint left_wheel_joint: axis 0 0 1 -> 0 0 -1; origin xyz=0.0 0.28 0 rpy=-1.5708 0 0 -> xyz=-0.3 0.35 0 rpy=1.5708 0 0
- joint line_left_joint: origin xyz=0.3 0.015 -0.12 -> xyz=0.45 0.035 -0.12
- joint line_right_joint: origin xyz=0.3 -0.015 -0.12 -> xyz=0.45 -0.035 -0.12
- joint right_wheel_joint: axis 0 0 1 -> 0 0 -1; origin xyz=0.0 -0.28 0 rpy=-1.5708 0 0 -> xyz=-0.3 -0.35 0 rpy=1.5708 0 0
